Commit message: Phase 1: Add RGBD camera to simulated robot
Add camera_link, camera_color_optical_frame, camera_depth_optical_frame
links with Gazebo Ignition rgbd_camera sensor (640x480, 15Hz, 60deg FOV).
Mount position and optical frame rotations match the real Orbbec Femto Bolt
hardware URDF. Bridge camera topics to ROS2 via ros_gz_bridge with
remappings to match real robot topic names.

File: src/rc_model_description/urdf/joints.xacro (robot description, xacro)
@@ -44,4 +44,20 @@
         <parent link="chassis_link"/>
         <child link="lidar_link"/>
+    </joint>
+    <!-- Camera mount (matches rc_model_hardware.urdf.xacro) -->
+    <joint name="camera_joint" type="fixed">
+        <origin xyz="0.0 0.05 0.08" rpy="0 0 -1.5707"/>
+        <parent link="chassis_link"/>
+        <child link="camera_link"/>
+    </joint>
+    <joint name="camera_depth_optical_joint" type="fixed">
+        <origin xyz="0 0 0" rpy="-1.5707 0 -1.5707"/>
+        <parent link="camera_link"/>
+        <child link="camera_depth_optical_frame"/>
+    </joint>
+    <joint name="camera_color_optical_joint" type="fixed">
+        <origin xyz="0 0 0" rpy="-1.5707 0 -1.5707"/>
+        <parent link="camera_link"/>
+        <child link="camera_color_optical_frame"/>
     </joint>
     <joint name="Rigid_278" type="fixed">

File: src/rc_model_description/urdf/links.xacro (robot description, xacro)
@@ -202,4 +202,41 @@
       </sensor>
     </gazebo>
+    <!-- ============================================================
+         RGBD Camera (matches Orbbec Femto Bolt on real robot)
+         Sensor attached to camera_link; optical frames rotate into
+         the standard camera convention (Z-forward, X-right, Y-down).
+         ============================================================ -->
+    <link name="camera_link">
+        <visual>
+            <origin xyz="0 0 0" rpy="0 0 0"/>
+            <geometry>
+                <box size="0.03 0.09 0.03"/>
+            </geometry>
+            <material name="black"/>
+        </visual>
+    </link>
+    <link name="camera_color_optical_frame"/>
+    <link name="camera_depth_optical_frame"/>
+    <gazebo reference="camera_link">
+      <sensor name="rgbd_camera" type="rgbd_camera">
+        <pose>0 0 0 0 0 0</pose>
+        <topic>camera</topic>
+        <update_rate>15</update_rate>
+        <camera>
+          <horizontal_fov>1.047</horizontal_fov>
+          <image>
+            <width>640</width>
+            <height>480</height>
+          </image>
+          <clip>
+            <near>0.1</near>
+            <far>10.0</far>
+          </clip>
+        </camera>
+        <always_on>true</always_on>
+        <visualize>true</visualize>
+        <gz_frame_id>camera_color_optical_frame</gz_frame_id>
+      </sensor>
+    </gazebo>
     <link name="servo">
         <inertial>
